File: TouchController.kicad_pcb (KiCad board)
At the start: 2 copper layers, 31 x 45 mm, 43 parts, among them J1 USB_B_Micro, J2 Connector, U1 TTP223, U2 TTP223, U3 TTP223, U4 TTP223, U5 TTP223, U6 TTP223, U7 TTP223, U8 TTP223, U9 NJM2884U1

Commit message: 基板 V1.1
Parts:
- removed D9: SchottkyDiode, TouchController:D_TUMD2
- moved F1 1.50 mm to (6.40, -5.40), turned to 180 degrees
- moved L1 1.50 mm to (6.40, -6.90), turned to 180 degrees
Connections:
- J1 pad 2: (no net) -> Net-(J1-Pad2)
- J1 pad 3: (no net) -> Net-(J1-Pad3)
- J1 pad 4: (no net) -> Net-(J1-Pad4)
- L1 pad 2: Net-(D9-Pad2) -> +5V
- U1 pad 6: (no net) -> Net-(U1-Pad6)
- U2 pad 6: (no net) -> Net-(U2-Pad6)
- U3 pad 6: (no net) -> Net-(U3-Pad6)
- U4 pad 6: (no net) -> Net-(U4-Pad6)
- U5 pad 4: (no net) -> Net-(U5-Pad4)
- U5 pad 6: (no net) -> Net-(U5-Pad6)
- U6 pad 4: (no net) -> Net-(U6-Pad4)
- U6 pad 6: (no net) -> Net-(U6-Pad6)
- U7 pad 6: (no net) -> Net-(U7-Pad6)
- U8 pad 6: (no net) -> Net-(U8-Pad6)
- U9 pad 3: (no net) -> Net-(U9-Pad3)
Routing:
- net GND: track 93.3 -> 95.5 mm, vias 11 -> 12
- net Net-(D9-Pad2): track 1.68 -> 0.00 mm
Other:
- board text added: "Touch Controller V1.1"
- board text removed: "Touch Controller V1.0"
